File: schema/schema.kicad_pcb (KiCad board)
At the start: 2 copper layers, 69 x 55.5 mm, 10 parts, among them J1 Autocom2, U4 LM7805_TO220

Commit message: finitions routage
Parts:
- moved C2 5.00 mm to (162.0, 91.0)
Routing:
- net Net-(J1-Pin_1): track 189.6 -> 255.9 mm
- net Net-(A1-+5V): track 129.0 -> 131.0 mm
- net Net-(U1-Vs): track 48.8 -> 50.5 mm
