File: schema/schema.kicad_pcb (KiCad board)
At the start: 2 copper layers, 69 x 55.5 mm, 10 parts, among them J1 Autocom2, U4 LM7805_TO220

Commit message: debut de code
Parts:
- C1: value C -> 330n
- C2: value C -> 100n
Changed lines of the file:
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@@
 		(tenting front back)
 		(pcbplotparams
-			(layerselection 0x00000000_00000000_55555555_5755f5ff)
+			(layerselection 0x00000000_00000000_55555555_57555551)
 			(plot_on_all_layers_selection 0x00000000_00000000_00000000_00000000)
 			(disableapertmacros no)
 			(usegerberextensions no)
-			(usegerberattributes yes)
-			(usegerberadvancedattributes yes)
-			(creategerberjobfile yes)
+			(usegerberattributes no)
+			(usegerberadvancedattributes no)
+			(creategerberjobfile no)
 			(dashed_line_dash_ratio 12.000000)
 			(dashed_line_gap_ratio 3.000000)
@@
 			(outputformat 1)
 			(mirror no)
-			(drillshape 1)
+			(drillshape 0)
 			(scaleselection 1)
-			(outputdirectory "")
+			(outputdirectory "output")
 		)
 	)
@@
 			)
 		)
-		(property "Value" "C"
+		(property "Value" "330n"
 			(at 2.5 2.5 0)
 			(layer "F.Fab")
@@
 			)
 		)
-		(property "Value" "C"
+		(property "Value" "100n"
 			(at 2.5 2.5 90)
 			(layer "F.Fab")
