File: schema/schema.kicad_sch (KiCad schematic)
At the start: 10 parts, among them J1 Conn_01x02_Pin, U4 LM7805_TO220

Commit message: debut de code
Parts:
- C1: value C -> 330n
- C2: value C -> 100n
- U4: footprint FootprintGamelGe2_v8.0:TO-220-3_Vertical -> FootprintGamelGe2_v8.0:TO-220-3_Horizontal_TabDown
Connections:
- net +5V: now reaches A1.5 (+5V), C2.1, R1.2, R2.2, U1.2 (Vcc), U2.2 (Vcc), U3.2 (Vcc), U4.3 (VO)
- net GND: now reaches A1.29 (GND), A1.6 (GND), A1.7 (GND), C1.2, C2.2, J1.2 (Pin_2), U1.3 (GND), U2.3 (GND), U3.3 (GND), U4.2 (GND)
Changed lines of the file:
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@@
+	)
+	(junction
+		(at 146.05 82.55)
+		(diameter 0)
+		(color 0 0 0 0)
 	)
 	(junction
@@
 	)
 	(junction
+		(at 179.07 71.12)
+		(diameter 0)
+		(color 0 0 0 0)
+	)
+	(junction
 		(at 149.86 130.81)
 		(diameter 0)
@@
 	(wire
 		(pts
-			(xy 195.58 71.12) (xy 170.18 71.12)
+			(xy 195.58 71.12) (xy 179.07 71.12)
 		)
 		(stroke
@@
 	(wire
 		(pts
+			(xy 146.05 82.55) (xy 149.86 82.55)
+		)
+		(stroke
+			(width 0)
+			(type default)
+		)
+	)
+	(wire
+		(pts
 			(xy 146.05 125.73) (xy 166.37 125.73)
 		)
@@
 	(wire
 		(pts
+			(xy 179.07 71.12) (xy 170.18 71.12)
+		)
+		(stroke
+			(width 0)
+			(type default)
+		)
+	)
+	(wire
+		(pts
 			(xy 146.05 99.06) (xy 149.86 99.06)
 		)
@@
 	(wire
 		(pts
-			(xy 138.43 82.55) (xy 149.86 82.55)
+			(xy 138.43 82.55) (xy 146.05 82.55)
 		)
 		(stroke
@@
 			)
 		)
-		(property "Value" "C"
+		(property "Value" "100n"
 			(at 168.91 77.4699 0)
 			(effects
@@
 	)
 	(symbol
+		(lib_id "power:GND")
+		(at 146.05 82.55 0)
+		(unit 1)
+		(exclude_from_sim no)
+		(in_bom yes)
+		(on_board yes)
+		(dnp no)
+		(fields_autoplaced yes)
+		(property "Reference" "#PWR01"
+			(at 146.05 88.9 0)
+			(effects
+				(font
+					(size 1.27 1.27)
+				)
+				(hide yes)
+			)
+		)
+		(property "Value" "GND"
+			(at 146.05 87.63 0)
+			(effects
+				(font
+					(size 1.27 1.27)
+				)
+			)
+		)
+		(property "Footprint" ""
+			(at 146.05 82.55 0)
+			(effects
+				(font
+					(size 1.27 1.27)
+				)
+				(hide yes)
+			)
+		)
+		(property "Datasheet" ""
+			(at 146.05 82.55 0)
+			(effects
+				(font
+					(size 1.27 1.27)
+				)
+				(hide yes)
+			)
+		)
+		(property "Description" "Power symbol creates a global label with name \"GND\" , ground"
+			(at 146.05 82.55 0)
+			(effects
+				(font
+					(size 1.27 1.27)
+				)
+				(hide yes)
+			)
+		)
+		(pin "1"
+		)
+		(instances
+			(project ""
+				(path "/9a88feef-e625-4185-af2b-8539e6f38877"
+					(reference "#PWR01")
+					(unit 1)
+				)
+			)
+		)
+	)
+	(symbol
 		(lib_id "Device:R")
 		(at 156.21 95.25 0)
@@
 			)
 		)
-		(property "Footprint" "FootprintGamelGe2_v8.0:TO-220-3_Vertical"
+		(property "Footprint" "FootprintGamelGe2_v8.0:TO-220-3_Horizontal_TabDown"
 			(at 153.67 65.405 0)
 			(effects
@@
 				(path "/9a88feef-e625-4185-af2b-8539e6f38877"
 					(reference "U4")
+					(unit 1)
+				)
+			)
+		)
+	)
+	(symbol
+		(lib_id "power:+5V")
+		(at 179.07 71.12 0)
+		(unit 1)
+		(exclude_from_sim no)
+		(in_bom yes)
+		(on_board yes)
+		(dnp no)
+		(fields_autoplaced yes)
+		(property "Reference" "#PWR02"
+			(at 179.07 74.93 0)
+			(effects
+				(font
+					(size 1.27 1.27)
+				)
+				(hide yes)
+			)
+		)
+		(property "Value" "+5V"
+			(at 179.07 66.04 0)
+			(effects
+				(font
+					(size 1.27 1.27)
+				)
+			)
+		)
+		(property "Footprint" ""
+			(at 179.07 71.12 0)
+			(effects
+				(font
+					(size 1.27 1.27)
+				)
+				(hide yes)
+			)
+		)
+		(property "Datasheet" ""
+			(at 179.07 71.12 0)
+			(effects
+				(font
+					(size 1.27 1.27)
+				)
+				(hide yes)
+			)
+		)
+		(property "Description" "Power symbol creates a global label with name \"+5V\""
+			(at 179.07 71.12 0)
+			(effects
+				(font
+					(size 1.27 1.27)
+				)
+				(hide yes)
+			)
+		)
+		(pin "1"
+		)
+		(instances
+			(project ""
+				(path "/9a88feef-e625-4185-af2b-8539e6f38877"
+					(reference "#PWR02")
 					(unit 1)
 				)
@@
 			)
 		)
-		(property "Value" "C"
+		(property "Value" "330n"
 			(at 142.24 77.4699 0)
 			(effects

Commit message: rangement du schema electronique
Parts:
- A1: value Arduino_UNO_R3 -> STM32F746
Connections:
- net +5V: now also A1.14 (SCL/A5), A1.31 (SDA/A4), R1.1, U1.1 (Vs), U3.1 (Signal)
Other:
- moved on the sheet: C1, C2, J1, R1, R2, U1, U2, U3, U4

Commit message: écriture des Readme
Other:
- title: (none) -> Schéma pour projet parking
Changed lines of the file:
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@@
 	(generator_version "9.0")
 	(paper "A4")
+	(title_block
+		(title "Schéma pour projet parking")
+		(date "25/05/2026")
+		(comment 1 "Marion Normand ")
+	)
 	(rectangle
 		(start 123.19 95.25)
